File: SolarSynth_digilog_THT/SolarSynth_THT.kicad_sch (KiCad schematic)
At the start: 31 parts, among them J1 OutputJack1, J2 Conn_01x01_Pin, J3 Conn_01x01_Pin, P1 PiezoDisc, P2 PiezoDisc, U1 74HC14, U2 MCP6002-xMC

Commit message: fixed some errors. Made it easier to solder and added blinkyparts logo
Parts:
- C1, C2, C3: footprint Capacitor_THT:C_Disc_D5.0mm_W2.5mm_P5.00mm -> blinkyparts:C_Disc_D5.0mm_W2.5mm_P5.00mm_handsoldering
Changed lines of the file:
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@@
 			)
 		)
-		(property "Footprint" "Capacitor_THT:C_Disc_D5.0mm_W2.5mm_P5.00mm"
+		(property "Footprint" "blinkyparts:C_Disc_D5.0mm_W2.5mm_P5.00mm_handsoldering"
 			(at 138.43 99.3648 0)
 			(effects
@@
 			)
 		)
-		(property "Footprint" "Capacitor_THT:C_Disc_D5.0mm_W2.5mm_P5.00mm"
+		(property "Footprint" "blinkyparts:C_Disc_D5.0mm_W2.5mm_P5.00mm_handsoldering"
 			(at 72.39 99.3648 0)
 			(effects
@@
 			)
 		)
-		(property "Footprint" "Capacitor_THT:C_Disc_D5.0mm_W2.5mm_P5.00mm"
+		(property "Footprint" "blinkyparts:C_Disc_D5.0mm_W2.5mm_P5.00mm_handsoldering"
 			(at 210.82 99.3648 0)
 			(effects
